Commit message: edjust lidar location

File: phoenixbot_description/urdf/groundbot/phoenixbot.xacro (robot description, xacro)
@@ -12,5 +12,5 @@
     <!-- ydlidar -->
     <xacro:ydlidar_sensor parent="chassis">
-        <origin xyz="0.0 0 0.22" rpy="0 0 0" />
+        <origin xyz="0.49 0.0 0.3" rpy="0 0 0" />
     </xacro:ydlidar_sensor>
     <!-- gps -->

File: phoenixbot_description/urdf/groundbot/ydlidar.xacro (robot description, xacro)
@@ -51,8 +51,8 @@
           <scan>
             <horizontal>
-              <samples>400</samples>
+              <samples>683</samples>
               <resolution>1</resolution>
-              <min_angle>-3.14159</min_angle>
-              <max_angle>3.14159</max_angle>
+              <min_angle>-2.0944</min_angle>
+              <max_angle>2.0944</max_angle>
             </horizontal>
           </scan>
